File: Test_Board.kicad_pcb (KiCad board)
At the start: 4 copper layers, 124 x 59 mm, 344 parts, among them J1 Conn_02x03_Counter_Clockwise, J43 USB_C_Receptacle, Q1 NPN, SW1 SW_Push, SW2 SW_Push, U1 STM32F103CBTx, U2 STM32G474QETx, U3 LD1117S33TR_SOT223, U5 SRV05-4, U6 STM32WB1MMCH6TR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

Commit message: PCB files to review
Parts:
- added REF**: MountingHole_2.7mm, MountingHole:MountingHole_2.7mm, F.Cu at (144.0, 74.8)
- added REF**: MountingHole_2.7mm, MountingHole:MountingHole_2.7mm, F.Cu at (28.5, 75.8)
- moved C4 1.92 mm to (136.6, 78.8)
- moved C6 1.92 mm to (139.4, 80.6)
- moved Y1 1.92 mm to (139.0, 77.8)
- moved R1 0.56 mm to (131.5, 120.0)
- moved R2 0.56 mm to (131.5, 121.0)
- moved C1 0.53 mm to (130.8, 122.5)
- moved C34 0.50 mm to (60.5, 111.0)
- moved C44 0.50 mm to (84.2, 104.8)
- moved D28 0.32 mm to (52.6, 80.5), turned to 180 degrees
- moved C28 0.27 mm to (70.2, 90.0)
- moved R40 0.17 mm to (52.5, 82.8), turned to 180 degrees
- moved C24 0.15 mm to (52.5, 81.8), turned to 180 degrees
Connections:
- C2 pad 1: (no net) -> +3V3
- C28 pad 1: (no net) -> +3V3
- C29 pad 1: (no net) -> +3V3
- C3 pad 1: (no net) -> +3V3
- C30 pad 1: (no net) -> +3V3
- C31 pad 1: (no net) -> +3V3
- C32 pad 1: (no net) -> +3V3
- C33 pad 1: (no net) -> +3V3
- C34 pad 1: (no net) -> +3V3
- C45 pad 1: (no net) -> +3V3
- C52 pad 1: (no net) -> +3V3
- C60 pad 1: (no net) -> +3V3
- C61 pad 1: (no net) -> +3V3
- C62 pad 1: (no net) -> +3V3
- C63 pad 1: (no net) -> +3V3
- D4 pad 1: (no net) -> +3V3
- EMG_UART1 pad 1: (no net) -> +3V3
- FB1 pad 2: (no net) -> +3V3
- Hapt_UART1 pad 1: (no net) -> +3V3
- J1 pad 1: (no net) -> +3V3
- Power1 pad 4: (no net) -> +3V3
- Q1 pad 1: (no net) -> +3V3
- R11 pad 2: (no net) -> +3V3
- R134 pad 1: (no net) -> +3V3
- R135 pad 1: (no net) -> +3V3
- R14 pad 1: (no net) -> +3V3
- R15 pad 2: (no net) -> +3V3
- R60 pad 2: (no net) -> +3V3
- RED1 pad 2: (no net) -> +3V3
- SW2 pad 1: (no net) -> +3V3
- U1 pad 1: (no net) -> +3V3
- U1 pad 24: (no net) -> +3V3
- U1 pad 36: (no net) -> +3V3
- U1 pad 48: (no net) -> +3V3
- U1 pad 9: (no net) -> +3V3
- U2 pad 128: (no net) -> +3V3
- U2 pad 13: (no net) -> +3V3
- U2 pad 24: Anlg_6 -> FSR1
- U2 pad 25: FSR1 -> FSR2
- U2 pad 26: FSR2 -> Anlg_6
- U2 pad 31: (no net) -> +3V3
- U2 pad 47: (no net) -> +3V3
- U2 pad 6: (no net) -> +3V3
- U2 pad 64: (no net) -> +3V3
- U2 pad 79: (no net) -> +3V3
- U2 pad 95: (no net) -> +3V3
- U3 pad 2: (no net) -> +3V3
- U6 pad 16: (no net) -> +3V3
- Y1 pad 2: (no net) -> +3V3
Routing:
- net +3V3: track 459.3 -> 302.2 mm
- net (no net): track 0.00 -> 59.1 mm
- net Anlg_6: track 20.4 -> 30.8 mm, vias 0 -> 2
- net VBUS: track 39.4 -> 45.2 mm
- net /Custom-debugger/D-: track 43.3 -> 47.6 mm
- net GND: track 197.9 -> 201.6 mm, vias 100 -> 101
- net FSR2: track 25.7 -> 27.8 mm
- net FSR1: track 26.0 -> 24.9 mm
- net /Custom-debugger/D+: track 50.7 -> 50.0 mm
- net Net-(U1-PD0): track 10.0 -> 9.43 mm

Commit message: PCB file reviewed
Parts:
- removed C10, C11, C12, C18, C19, C20, C21, C22, C23, C24, C25, C26, C35, C36, C37, C38, C39, C40, C41, C42, C53, C7, C8, C9: 4.7n, Capacitor_SMD:C_0402_1005Metric
- removed D53: PESD5V0L1UL, Diode_SMD:D_SOD-882
- added D48: PESD5V0L1UL, Diode_SMD:D_SOD-882, F.Cu at (33.2, 84.3)
- C13, C14, C15, C16, C17, C27: value 4.7n -> 1u
- R129, R17, R25, R26, R27, R28, R34, R35, R36, R37, R38, R39, R40, R41, R42, R51, R52, R53, R54, R55, R56, R57, R58, R64: value 1k -> 47
- moved D45 2.95 mm to (33.2, 87.3), turned to 90 degrees
- moved D41 2.65 mm to (33.2, 97.2), turned to 90 degrees
- moved D43 2.50 mm to (33.2, 92.2), turned to 90 degrees
- moved D40 2.35 mm to (33.2, 99.6), turned to -90 degrees
- moved D44 2.30 mm to (33.2, 89.7), turned to -90 degrees
- moved D42 2.25 mm to (33.2, 94.3), turned to -90 degrees
- moved R34 1.11 mm to (34.5, 115.5)
- moved R54 1.08 mm to (34.5, 94.8)
- moved R53 1.08 mm to (34.5, 97.0)
- moved R39 1.06 mm to (34.5, 104.8)
- moved R41 1.06 mm to (54.8, 81.8)
- moved R55 1.04 mm to (34.5, 92.0)
- moved R52 1.03 mm to (34.5, 99.8)
- moved R56 1.03 mm to (34.5, 89.8)
- moved R57 1.03 mm to (34.5, 87.2)
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- renumbered RED1 to BLUE1, RED2 to BLUE2
Connections:
- Ecod1 pad 2: Net-(D53-K) -> Net-(D40-K)
- Ecod1 pad 3: Net-(D40-K) -> Net-(D41-K)
- Ecod1 pad 4: Net-(D41-K) -> Net-(D42-K)
- Ecod1 pad 5: Net-(D42-K) -> Net-(D43-K)
- Ecod1 pad 6: Net-(D43-K) -> Net-(D44-K)
- Ecod1 pad 7: Net-(D44-K) -> Net-(D45-K)
- Ecod1 pad 8: Net-(D45-K) -> Net-(D48-K)
- R52 pad 1: Net-(D53-K) -> Net-(D40-K)
- R53 pad 1: Net-(D40-K) -> Net-(D41-K)
- R54 pad 1: Net-(D41-K) -> Net-(D42-K)
- R55 pad 1: Net-(D42-K) -> Net-(D43-K)
- R56 pad 1: Net-(D43-K) -> Net-(D44-K)
- R57 pad 1: Net-(D44-K) -> Net-(D45-K)
- R58 pad 1: Net-(D45-K) -> Net-(D48-K)
Routing:
- net GND: track 201.6 -> 183.4 mm
- net Net-(D53-K): track 6.65 -> 0.00 mm
- net Net-(D48-K): track 0.00 -> 5.52 mm
- net Net-(D42-K): track 7.61 -> 5.21 mm
- net Net-(D44-K): track 7.15 -> 5.31 mm
- net Net-(D40-K): track 7.00 -> 5.24 mm
- net Net-(Curr1-Pin_1): track 6.60 -> 5.25 mm
- net Anlg_1: track 33.2 -> 34.4 mm
- net Net-(Analog6-8-Pin_2): track 7.06 -> 5.92 mm
- net Net-(Curr1-Pin_7): track 6.56 -> 5.44 mm
- net Ecod_6: track 34.6 -> 35.7 mm
- net Ecod_2: track 29.7 -> 30.8 mm
- net Ecod_7: track 33.7 -> 34.8 mm
- net Curr1: track 14.7 -> 15.8 mm
- net Net-(Analog1-5-Pin_1): track 6.99 -> 5.90 mm
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Other:
- board size 124 x 59 mm -> 124.5 x 59 mm
